File: board/MainBoard.brd (EAGLE design)
At the start: 63.2 x 82.5 mm, 85 parts, among them IC1 MAX481CSA, IC3 MAX481CSA, U1 6N137S, U12 OSCILLATORSMD, U2 6N137S, U3 6N137S, U4 6N137S, U5 6N137S, U6 6N137S, U7 LAN8720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

Commit message: ftp temp commit
Parts:
- C4: value 22uF -> 0.22uF
- C7: value (none) -> 0.1
- LED1, LED2: value (none) -> green
- R21, R22, R23, R24: value 49.9k 1% -> 49.9 1%
- R3, R36: value 1.5k -> 4.7k
Connections:
- net CRYSTAL_OUT: now also U12.P$3
- net GPIO0: no longer U12.P$3
Routing:
- net GPIO0: track 48.6 -> 45.2 mm
